File: prototype_schematics/prototype-filter.kicad_pcb (KiCad board)
At the start: 2 copper layers, 24.4 x 22.9 mm, 6 parts, among them J1 Conn_Coaxial, J2 Conn_Coaxial, J3 Conn_Coaxial, J4 Conn_Coaxial, U1 TA0411A, Y1 Resonator

Commit message: adding filters and amps
Changed lines of the file:
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@@
       (drillshape 0)
       (scaleselection 1)
-      (outputdirectory "")
+      (outputdirectory "gerbers")
     )
   )
@@
     )
     (fp_line (start -2.54003 -2.540005) (end -2.121158 -2.540005)
-      (stroke (width 0.254) (type solid)) (layer "F.SilkS"))
+      (stroke (width 0.254001) (type solid)) (layer "F.SilkS"))
     (fp_line (start -2.54003 -0.65113) (end -2.54003 -2.540005)
-      (stroke (width 0.254) (type solid)) (layer "F.SilkS"))
+      (stroke (width 0.254001) (type solid)) (layer "F.SilkS"))
     (fp_line (start -2.54003 2.540005) (end -2.54003 0.65113)
-      (stroke (width 0.254) (type solid)) (layer "F.SilkS"))
+      (stroke (width 0.254001) (type solid)) (layer "F.SilkS"))
     (fp_line (start -2.121158 2.540005) (end -2.54003 2.540005)
-      (stroke (width 0.254) (type solid)) (layer "F.SilkS"))
+      (stroke (width 0.254001) (type solid)) (layer "F.SilkS"))
     (fp_line (start 1.721107 -2.540005) (end 2.53998 -2.540005)
-      (stroke (width 0.254) (type solid)) (layer "F.SilkS"))
+      (stroke (width 0.254001) (type solid)) (layer "F.SilkS"))
     (fp_line (start 2.53998 -2.540005) (end 2.53998 -0.523673)
-      (stroke (width 0.254) (type solid)) (layer "F.SilkS"))
+      (stroke (width 0.254001) (type solid)) (layer "F.SilkS"))
     (fp_line (start 2.53998 0.523673) (end 2.53998 2.540005)
-      (stroke (width 0.254) (type solid)) (layer "F.SilkS"))
+      (stroke (width 0.254001) (type solid)) (layer "F.SilkS"))
     (fp_line (start 2.53998 2.540005) (end 1.721107 2.540005)
-      (stroke (width 0.254) (type solid)) (layer "F.SilkS"))
+      (stroke (width 0.254001) (type solid)) (layer "F.SilkS"))
     (fp_circle (center -2.74003 2.667005) (end -2.710033 2.667005)
       (stroke (width 0.059995) (type solid)) (fill none) (layer "F.SilkS"))
