File: aprs_receiver_board/aprs_receiver_board/power.kicad_sch (KiCad schematic)
At the start: 13 parts, among them U4 LP38693MP-3.3

Commit message: Add decoupling capacitor and IO connectors
Parts:
- F1: footprint (none) -> Fuse:Fuse_1206_3216Metric_Pad1.42x1.75mm_HandSolder
- TP6: renamed from TP1; footprint (none) -> TestPoint:TestPoint_Keystone_5000-5004_Miniature
- TP7: renamed from TP2; footprint (none) -> TestPoint:TestPoint_Keystone_5000-5004_Miniature
- TP8: renamed from TP3; footprint (none) -> TestPoint:TestPoint_Keystone_5000-5004_Miniature
- TP9: renamed from TP4; footprint (none) -> TestPoint:TestPoint_Keystone_5000-5004_Miniature
- renumbered R12 to R7, R11 to R8, R13 to R9, U4 to U3
Changed lines of the file:
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@@
 		(dnp no)
 		(fields_autoplaced yes)
-		(property "Reference" "#PWR054"
+		(property "Reference" "#PWR031"
 			(at 196.85 31.75 0)
 			(effects
@@
 			(project "aprs_receiver_board"
 				(path "/8a8e4ede-5ef9-4a53-a3a5-89928e3630c6/3e24cd22-99b8-4f24-a536-e33a1068bbd2"
-					(reference "#PWR054")
+					(reference "#PWR031")
 					(unit 1)
 				)
@@
 		(dnp no)
 		(fields_autoplaced yes)
-		(property "Reference" "#PWR050"
+		(property "Reference" "#PWR028"
 			(at 128.27 53.34 0)
 			(effects
@@
 			(project "aprs_receiver_board"
 				(path "/8a8e4ede-5ef9-4a53-a3a5-89928e3630c6/3e24cd22-99b8-4f24-a536-e33a1068bbd2"
-					(reference "#PWR050")
+					(reference "#PWR028")
 					(unit 1)
 				)
@@
 		(dnp no)
 		(fields_autoplaced yes)
-		(property "Reference" "R12"
+		(property "Reference" "R7"
 			(at 55.88 40.6399 0)
 			(effects
@@
 			(project "aprs_receiver_board"
 				(path "/8a8e4ede-5ef9-4a53-a3a5-89928e3630c6/3e24cd22-99b8-4f24-a536-e33a1068bbd2"
-					(reference "R12")
+					(reference "R7")
 					(unit 1)
 				)
@@
 		(dnp no)
 		(fields_autoplaced yes)
-		(property "Reference" "#PWR056"
+		(property "Reference" "#PWR033"
 			(at 231.14 31.75 0)
 			(effects
@@
 			(project "aprs_receiver_board"
 				(path "/8a8e4ede-5ef9-4a53-a3a5-89928e3630c6/3e24cd22-99b8-4f24-a536-e33a1068bbd2"
-					(reference "#PWR056")
+					(reference "#PWR033")
 					(unit 1)
 				)
@@
 		(dnp no)
 		(fields_autoplaced yes)
-		(property "Reference" "#PWR049"
+		(property "Reference" "#PWR025"
 			(at 85.09 53.34 0)
 			(effects
@@
 			(project "aprs_receiver_board"
 				(path "/8a8e4ede-5ef9-4a53-a3a5-89928e3630c6/3e24cd22-99b8-4f24-a536-e33a1068bbd2"
-					(reference "#PWR049")
+					(reference "#PWR025")
 					(unit 1)
 				)
@@
 		(dnp no)
 		(fields_autoplaced yes)
-		(property "Reference" "#PWR055"
+		(property "Reference" "#PWR032"
 			(at 214.63 31.75 0)
 			(effects
@@
 			(project "aprs_receiver_board"
 				(path "/8a8e4ede-5ef9-4a53-a3a5-89928e3630c6/3e24cd22-99b8-4f24-a536-e33a1068bbd2"
-					(reference "#PWR055")
+					(reference "#PWR032")
 					(unit 1)
 				)
@@
 		(dnp no)
 		(fields_autoplaced yes)
-		(property "Reference" "TP4"
+		(property "Reference" "TP9"
 			(at 248.92 33.7819 0)
 			(effects
@@
 			)
 		)
-		(property "Footprint" ""
+		(property "Footprint" "TestPoint:TestPoint_Keystone_5000-5004_Miniature"
 			(at 241.3 31.75 0)
 			(effects
@@
 			(project "aprs_receiver_board"
 				(path "/8a8e4ede-5ef9-4a53-a3a5-89928e3630c6/3e24cd22-99b8-4f24-a536-e33a1068bbd2"
-					(reference "TP4")
+					(reference "TP9")
 					(unit 1)
 				)
@@
 		(dnp no)
 		(fields_autoplaced yes)
-		(property "Reference" "#PWR047"
+		(property "Reference" "#PWR027"
 			(at 128.27 30.48 0)
 			(effects
@@
 			(project "aprs_receiver_board"
 				(path "/8a8e4ede-5ef9-4a53-a3a5-89928e3630c6/3e24cd22-99b8-4f24-a536-e33a1068bbd2"
-					(reference "#PWR047")
+					(reference "#PWR027")
 					(unit 1)
 				)
@@
 		(dnp no)
 		(fields_autoplaced yes)
-		(property "Reference" "#PWR053"
+		(property "Reference" "#PWR030"
 			(at 157.48 53.34 0)
 			(effects
@@
 			(project "aprs_receiver_board"
 				(path "/8a8e4ede-5ef9-4a53-a3a5-89928e3630c6/3e24cd22-99b8-4f24-a536-e33a1068bbd2"
-					(reference "#PWR053")
+					(reference "#PWR030")
 					(unit 1)
 				)
@@
 		(dnp no)
 		(fields_autoplaced yes)
-		(property "Reference" "R11"
+		(property "Reference" "R8"
 			(at 95.25 33.0199 0)
 			(effects
@@
 			(project "aprs_receiver_board"
 				(path "/8a8e4ede-5ef9-4a53-a3a5-89928e3630c6/3e24cd22-99b8-4f24-a536-e33a1068bbd2"
-					(reference "R11")
+					(reference "R8")
 					(unit 1)
 				)
@@
 		(dnp no)
 		(fields_autoplaced yes)
-		(property "Reference" "TP3"
+		(property "Reference" "TP8"
 			(at 233.68 33.7819 0)
 			(effects
@@
 			)
 		)
-		(property "Footprint" ""
+		(property "Footprint" "TestPoint:TestPoint_Keystone_5000-5004_Miniature"
 			(at 226.06 31.75 0)
 			(effects
@@
 			(project "aprs_receiver_board"
 				(path "/8a8e4ede-5ef9-4a53-a3a5-89928e3630c6/3e24cd22-99b8-4f24-a536-e33a1068bbd2"
-					(reference "TP3")
+					(reference "TP8")
 					(unit 1)
 				)
@@
 		(dnp no)
 		(fields_autoplaced yes)
-		(property "Reference" "#PWR057"
+		(property "Reference" "#PWR034"
 			(at 246.38 31.75 0)
 			(effects
@@
 			(project "aprs_receiver_board"
 				(path "/8a8e4ede-5ef9-4a53-a3a5-89928e3630c6/3e24cd22-99b8-4f24-a536-e33a1068bbd2"
-					(reference "#PWR057")
+					(reference "#PWR034")
 					(unit 1)
 				)
@@
 		(dnp no)
 		(fields_autoplaced yes)
-		(property "Reference" "#PWR052"
+		(property "Reference" "#PWR029"
 			(at 157.48 27.94 0)
 			(effects
@@
 			(project "aprs_receiver_board"
 				(path "/8a8e4ede-5ef9-4a53-a3a5-89928e3630c6/3e24cd22-99b8-4f24-a536-e33a1068bbd2"
-					(reference "#PWR052")
+					(reference "#PWR029")
 					(unit 1)
 				)
@@
 		(dnp no)
 		(fields_autoplaced yes)
-		(property "Reference" "R13"
+		(property "Reference" "R9"
 			(at 160.02 39.3699 0)
 			(effects
@@
 			(project "aprs_receiver_board"
 				(path "/8a8e4ede-5ef9-4a53-a3a5-89928e3630c6/3e24cd22-99b8-4f24-a536-e33a1068bbd2"
-					(reference "R13")
+					(reference "R9")
 					(unit 1)
 				)
@@
 		(dnp no)
 		(fields_autoplaced yes)
-		(property "Reference" "TP1"
+		(property "Reference" "TP6"
 			(at 199.39 33.7819 0)
 			(effects
@@
 			)
 		)
-		(property "Footprint" ""
+		(property "Footprint" "TestPoint:TestPoint_Keystone_5000-5004_Miniature"
 			(at 191.77 31.75 0)
 			(effects
@@
 			(project "aprs_receiver_board"
 				(path "/8a8e4ede-5ef9-4a53-a3a5-89928e3630c6/3e24cd22-99b8-4f24-a536-e33a1068bbd2"
-					(reference "TP1")
+					(reference "TP6")
 					(unit 1)
 				)
@@
 		(dnp no)
 		(fields_autoplaced yes)
-		(property "Reference" "TP2"
+		(property "Reference" "TP7"
 			(at 217.17 33.7819 0)
 			(effects
@@
 			)
 		)
-		(property "Footprint" ""
+		(property "Footprint" "TestPoint:TestPoint_Keystone_5000-5004_Miniature"
 			(at 209.55 31.75 0)
 			(effects
@@
 			(project "aprs_receiver_board"
 				(path "/8a8e4ede-5ef9-4a53-a3a5-89928e3630c6/3e24cd22-99b8-4f24-a536-e33a1068bbd2"
-					(reference "TP2")
+					(reference "TP7")
 					(unit 1)
 				)
@@
 		(dnp no)
 		(fields_autoplaced yes)
-		(property "Reference" "#PWR046"
+		(property "Reference" "#PWR024"
 			(at 85.09 30.48 0)
 			(effects
@@
 			(project "aprs_receiver_board"
 				(path "/8a8e4ede-5ef9-4a53-a3a5-89928e3630c6/3e24cd22-99b8-4f24-a536-e33a1068bbd2"
-					(reference "#PWR046")
+					(reference "#PWR024")
 					(unit 1)
 				)
@@
 			)
 		)
-		(property "Footprint" ""
+		(property "Footprint" "Fuse:Fuse_1206_3216Metric_Pad1.42x1.75mm_HandSolder"
 			(at 43.18 29.718 90)
 			(effects
@@
 		(dnp no)
 		(fields_autoplaced yes)
-		(property "Reference" "#PWR014"
+		(property "Reference" "#PWR022"
 			(at 53.34 30.48 0)
 			(effects
@@
 			(project "aprs_receiver_board"
 				(path "/8a8e4ede-5ef9-4a53-a3a5-89928e3630c6/3e24cd22-99b8-4f24-a536-e33a1068bbd2"
-					(reference "#PWR014")
+					(reference "#PWR022")
 					(unit 1)
 				)
@@
 		(dnp no)
 		(fields_autoplaced yes)
-		(property "Reference" "#PWR048"
+		(property "Reference" "#PWR026"
 			(at 110.49 53.34 0)
 			(effects
@@
 			(project "aprs_receiver_board"
 				(path "/8a8e4ede-5ef9-4a53-a3a5-89928e3630c6/3e24cd22-99b8-4f24-a536-e33a1068bbd2"
-					(reference "#PWR048")
+					(reference "#PWR026")
 					(unit 1)
 				)
@@
 		(dnp no)
 		(fields_autoplaced yes)
-		(property "Reference" "U4"
+		(property "Reference" "U3"
 			(at 110.49 24.13 0)
 			(effects
@@
 			(project "aprs_receiver_board"
 				(path "/8a8e4ede-5ef9-4a53-a3a5-89928e3630c6/3e24cd22-99b8-4f24-a536-e33a1068bbd2"
-					(reference "U4")
+					(reference "U3")
 					(unit 1)
 				)
@@
 		(dnp no)
 		(fields_autoplaced yes)
-		(property "Reference" "#PWR051"
+		(property "Reference" "#PWR023"
 			(at 53.34 53.34 0)
 			(effects
@@
 			(project "aprs_receiver_board"
 				(path "/8a8e4ede-5ef9-4a53-a3a5-89928e3630c6/3e24cd22-99b8-4f24-a536-e33a1068bbd2"
-					(reference "#PWR051")
-					(unit 1)
-				)
+					(reference "#PWR023")
+					(unit 1)
+				)
