File: aprs_receiver_board/aprs_receiver_board/usb_interface.kicad_sch (KiCad schematic)
At the start: 25 parts, among them J1 USB_B, U1 FT2232HL, U2 93LC56BT-I/OT, Y1 12 MHz

Commit message: Add decoupling capacitor and IO connectors
Parts:
- FB1, FB2: footprint (none) -> Resistor_SMD:R_0805_2012Metric_Pad1.20x1.40mm_HandSolder
- J1: footprint (none) -> Connector_USB:USB_B_OST_USB-B1HSxx_Horizontal
- TP1: renamed from TP5; footprint (none) -> TestPoint:TestPoint_Keystone_5000-5004_Miniature
- TP2: renamed from TP6; footprint (none) -> TestPoint:TestPoint_Keystone_5000-5004_Miniature
- TP3: renamed from TP7; footprint (none) -> TestPoint:TestPoint_Keystone_5000-5004_Miniature
- TP4: renamed from TP8; footprint (none) -> TestPoint:TestPoint_Keystone_5000-5004_Miniature
- TP5: renamed from TP9; footprint (none) -> TestPoint:TestPoint_Keystone_5000-5004_Miniature
- Y1: footprint (none) -> Crystal:Resonator-2Pin_W10.0mm_H5.0mm
- renumbered C8 to C1, C5 to C2, C7 to C3, C6 to C5, C1 to C6, C3 to C7, C2 to C8, R3 to R1, R1 to R2, R6 to R3, R5 to R4, R2 to R5, R4 to R6, U2 to U1, U1 to U2
Other:
- moved on the sheet: C1
